File: eagle_NAHS-LatchBrick/v1.0_r1.brd (EAGLE design)
At the start: 45.5 x 70.3 mm, 34 parts, among them IC1 ESP12F, IC2 TP4056, IC3 DW01A, IC4 FT232RL, IC5 ATTINY212-SSNR, J1 10118194-0001LF, Q1 8205A

Commit message: Board v1.0_R1 should allready be finished
Parts:
- added L1, L2: PINHD_1X02_R_1, no_pinhd:1X02_R_1
- added R12: 2.7M, rcl:R0805
- added R6: 3.9k, rcl:R0805
- IC2: value TP4056 -> ATTINY212-SSNR; device no_reichelt:SO8-THERMALPAD -> no_microchip:SOIC8
- IC3: value DW01A -> TP4056; device no_reichelt:SOT23-6 -> no_reichelt:SO8-THERMALPAD
- IC4: value FT232RL -> DW01A; device ftdichip:SSOP28 -> no_reichelt:SOT23-6
- IC5: value ATTINY212-SSNR -> FT232RL; device no_microchip:SOIC8 -> ftdichip:SSOP28
- R10: value 590k -> 10k
- R11: value 2.7M -> 590k
- R7: value 10k -> 3.9k
- moved IC2 30.9 mm to (35.6, 29.2), turned to 90 degrees
- moved IC5 29.2 mm to (35.6, 58.4)
- moved IC4 18.1 mm to (24.1, 44.5)
- moved IC3 14.0 mm to (25.4, 58.4), turned to 180 degrees
- moved R10 13.1 mm to (20.3, 22.9), turned to 0 degrees
- moved R8 6.35 mm to (20.3, 12.7)
- moved UPDI 4.66 mm to (25.9, 32.6)
- moved R11 4.32 mm to (24.1, 35.4)
- moved R7 1.27 mm to (20.3, 15.2)
- moved R9 1.27 mm to (20.3, 20.3)
Connections:
- removed net N$5: IC5.6, UPDI.1
- removed net N$6: C3.1, IC4.17, IC4.4
- new net L1: IC2.2, L1.1
- new net L2: IC2.3, L2.1
- new net UPDI: IC2.6, UPDI.1
- new net VCCIO: C3.1, IC5.17, IC5.4
- net +3V3: now also IC2.1, R6.1, R9.1; no longer IC5.1
- net A0: now also R11.1, R12.2; no longer R10.1, R11.2
- net BAT+: now also IC3.5; no longer IC2.5
- net BOOT1: now also R9.2; no longer R8.2
- net BOOT2: now also R10.2; no longer R9.2
- net CHRG: now also IC3.7; no longer IC2.7
- net D+: now also IC5.15; no longer IC4.15
- net D-: now also IC5.16; no longer IC4.16
- net EN: now also R8.2; no longer R7.2
- net GND: now also IC2.8, L1.2, L2.2, R10.1, R11.2; no longer IC5.8, R10.2, R9.1
- net IN+: now also IC5.20; no longer IC4.20
- net IN-: now also IC3.1, IC3.3, IC3.T1, IC3.T2, IC3.T3, IC3.T4, IC3.T5, IC3.T6, IC3.T7, IC3.T8, IC4.6, IC5.18, IC5.21, IC5.25, IC5.26, IC5.7; no longer IC2.1, IC2.3, IC2.T1, IC2.T2, IC2.T3, IC2.T4, IC2.T5, IC2.T6, IC2.T7, IC2.T8, IC3.6, IC4.18, IC4.21, IC4.25, IC4.26, IC4.7
- net N$1: now also IC3.4, IC3.8; no longer IC2.4, IC2.8
- net N$11: now also IC4.3; no longer IC3.3
- net N$2: now also IC3.2; no longer IC2.2
- net N$3: now also IC4.2; no longer IC3.2
- net N$4: now also IC4.5; no longer IC3.5
- net N$8: now also IC4.1; no longer IC3.1
- net RST: now also IC2.7; no longer IC5.7
- net RXD: now also IC5.1; no longer IC4.1
- net SCL: now also IC2.5, R7.2; no longer IC5.5
- net SDA: now also IC2.4, R6.2; no longer IC5.4
- net SEL+: now also R12.1; no longer R11.1
- net STDBY: now also IC3.6; no longer IC2.6
- net TXD: now also IC5.5; no longer IC4.5
Routing:
- net GND: track 51.5 -> 102.2 mm, vias 0 -> 1
- net +3V3: track 39.9 -> 81.6 mm
- net SDA: track 0.00 -> 34.5 mm, vias 0 -> 2
- net SCL: track 0.00 -> 33.8 mm, vias 0 -> 2
- net VCCIO: track 0.00 -> 23.3 mm, vias 0 -> 2
- net N$6: track 23.3 -> 0.00 mm, vias 2 -> 0
- net L2: track 0.00 -> 16.1 mm
- net L1: track 0.00 -> 10.7 mm
- net EN: track 31.7 -> 22.1 mm
- net UPDI: track 0.00 -> 8.21 mm
- net RST: track 57.3 -> 64.2 mm, vias 3 -> 4
- net A0: track 42.4 -> 41.1 mm
- net STDBY: track 54.9 -> 55.7 mm
- net CHRG: track 57.9 -> 58.7 mm
- net BOOT1: track 5.63 -> 6.15 mm
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Other:
- board text added: "NAHS-LatchBrick"
- board text added: "v1.0 R1"
- board text removed: "NAHS-TempBrick"
- board text removed: "v1.0 R2"
