File: eagle_NAHS-LatchBrick/v1.0_r3.sch (EAGLE design)
At the start: 38 parts, among them IC1 ESP12S, IC2 ATTINY212-SSNR, IC3 TP4056, IC4 DW01A, J1 10118194-0001LF, J2 BRICK-INTERF-V3_B-SIDE, Q1 8205A

Commit message: v1.0 R3 Board done
Parts:
- removed R15: 10k, rcl:R-EU_R0805
- removed R16: 590k, rcl:R-EU_R0805
- removed R17: 2.7M, rcl:R-EU_R0805
- added R3, R4, R5: 1k, rcl:R-EU_R0805
- R10, R11: value 3.9k -> 10k
- R13: value 10k -> 590k
- R14: value 10k -> 2.7M
- R6: value 1k -> 1.74k
- R7, R8: value 1k -> 3.9k
- R9: value 1.74k -> 10k
Connections:
- net +3V3: now also R7.1, R8.1, R9.1; no longer R11.1, R12.1, R13.1
- net A0: now also R13.1, R14.2; no longer R16.1, R17.2
- net BAT-: now also R3.1; no longer R6.1
- net BOOT1: now also R10.2; no longer R13.2
- net BOOT2: now also R11.2; no longer R14.2
- net CD: now also R12.2; no longer R15.2
- net CHRG: now also R4.2; no longer R7.2
- net EN: now also R9.2; no longer R12.2
- net GND: now also R11.1, R13.2; no longer R14.1, R16.2
- net IN-: now also R6.1; no longer R9.1
- net N$1: now also R12.1; no longer R15.1
- net N$2: now also R6.2; no longer R9.2
- net N$3: now also R3.2; no longer R6.2
- net N$7: now also R4.1; no longer R7.1
- net RST: now also R5.2; no longer R8.2
- net SCL: now also R8.2; no longer R11.2
- net SDA: now also R7.2; no longer R10.2
- net SEL+: now also R14.1; no longer R17.1
- net WAKE: now also R5.1; no longer R8.1
Other:
- moved on the sheet: R10, R11, R12, R13, R14, R6, R7, R8, R9
