File: kicad/nahs-LatchBrick_v1.0_r4/nahs-LatchBrick_v1.0_r4.kicad_pcb (KiCad board)
At the start: 2 copper layers, 49 x 74 mm, 63 parts, among them IC1 ESP12S, IC3 ATTINY414, J2 USB_B_Mini, Q1 8205A, Q3 CJ2302, Q4 MMBT2907A, SW1 KMR_231_G_LFS, SW2 SSSS820101, U1 ZD8028IB5TR, U3 DW01A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

Commit message: the firmware is now on the latest schema
Parts:
- J2: footprint Connector_USB:USB_Micro-B_Amphenol_10118194_Horizontal -> no_common:USB_Micro-B_Amphenol_10118194_Horizontal
